File: design_files/AST1004.sch (EAGLE design)
At the start: 11 parts, among them J1 SM05B, U1 TCS34725FN

Commit message: updated documentation
Parts:
- removed C4: 1uF, tinycircuits:AS-ITM-00105
- removed R4: 5.0, tinycircuits:AS-ITM-00289
- added C3: 0.1uF, tinycircuits:AS-ITM-00008
- C1: value 0.1uF -> 1uF; device tinycircuits:AS-ITM-00008 -> tinycircuits:AS-ITM-00105; PARTNO (none) -> AS-ITM-00105; VALUE (none) -> 1uF
- C2: value 10uF -> 1uF; device tinycircuits:AS-ITM-00002 -> tinycircuits:AS-ITM-00105; PARTNO (none) -> AS-ITM-00105; VALUE (none) -> 1uF
- D1, D2: value LED -> QBLP674-IWM-NW; device tinycircuits:AS-ITM-00049 -> tinycircuits:AS-ITM-00554; PARTNO AS-ITM-00049 -> AS-ITM-00554; VALUE 47uF -> QBLP674-IWM-NW
- J1: device tinycircuits:AS-ITM-00340 -> tinycircuits:AS-ITM-00340EDGE
- R1: value 10.0K -> 27.0; device tinycircuits:AS-ITM-00032 -> tinycircuits:AS-ITM-00240
- R2: value 27.0 -> 5K; device tinycircuits:AS-ITM-00240 -> tinycircuits:AS-ITM-00289
- R3: value 0.0 -> 5K; device tinycircuits:AS-ITM-00076 -> tinycircuits:AS-ITM-00289
Connections:
- removed net LDR: D1.2, D2.2, R4.2, U1.NC
- new net N$3: D2.C, R3.2
- new net N$4: D1.C, R2.2
- net GND: now also C3.2; no longer C4.2
- net INT: no longer R1.1, R3.2
- net N$1: now also R2.1; no longer R4.1
- net N$2: now also C2.1, C3.1, R1.2; no longer C1.1, C4.1, R2.2
- net VCC: now also C1.1, D1.A, D2.A, R1.1; no longer C2.1, D1.1, D2.1, R1.2, R2.1
Other:
- note added: "3"
- note added: "Non Populated: -"
- note added: "TCS34725 Color Sensor"
- note added: "Wireling Color Sensor"
- note removed: "*NC is LDR "IR LED Constant Current Sink" pin"
- note removed: "2"
- note removed: "Color Sensor = DigiKey: TCS37717FNCT-ND"
- note removed: "Color Sensor Board"
- note removed: "LED = DigiKey: 1516-1122-1-ND"
- note removed: "Non Populated: R1, R3"
- note removed: "TCS3771 Color Sensor"
- moved on the sheet: C1, C2, R1, R2, R3
